File: OCP-3/OCP-3.sch (KiCad schematic (older format))
At the start: 183 parts, among them X1 ico*отверстие*М3, X2 ico*отверстие*М3, X3 ico*отверстие*М3, X4 ico*отверстие*М3, X5 ico*LOGO_NIKITOS_10х10

Commit message: на схему вынесены транзисторы
Parts:
- removed C18, C19, C20, C21, C22, C23, C24, C25: Конденсатор*0,1мкФ*25В*0603, N_RLC:Конденсатор_SMD_IEC_0603, symbol eo-engine:Конденсатор*0,1мкФ*25В*0603
- removed R54, R55, R56, R57, R58, R59, R60, R61: Резистор*1кОм*0603, N_RLC:Резистор_SMD_0603_0,065_Вт_pnp, symbol eo-engine:Резистор*1кОм*0603
- removed VD34, VD35, VD36, VD37, VD38, VD39, VD40, VD41: Стабилитрон*3,9В*SOD80, N_VD_HL:SOD-80, symbol eo-engine:Стабилитрон*3,9В*SOD80
- removed XP16, XP17: Клеммник*шаг_3,5*5контактов*1ряд*вертикальная, N_X:Клеммник_15EDGVC-3.5-05P, symbol eo-engine:Клеммник*шаг_3,5*5контактов*1ряд*вертикальная
- added VT21, VT22, VT23, VT24, VT25, VT26, VT27, VT28: Транзистор_NPN_1Б-2(4)К-3Э_0, N_VD_HL:Транзистор_NPN_SOT223, symbol elements:Транзистор_NPN_1Б-2(4)К-3Э_0
Connections:
- net GND: now also XP18.5
- no-connect marks 7 -> 4
Other:
- note added: "h21=100"
- note added: "требуется:\n8 транзисторных выходов 6А (5 подсветка, 1 ТТР, 2 запас)\n2 механических реле\n4 дискретных входа"
- moved on the sheet: XP18
